Commit message: Sensors appear to be working

File: car/urdf/car.xacro (robot description, xacro)
@@ -371,4 +371,58 @@
             </collision>
         </link>
+	  <!-- Camera -->
+	  <joint name="camera_joint" type="fixed">
+	    <axis xyz="0 1 0" />
+	    <origin xyz="0.2 0.2 0.2" rpy="0 0 0"/>
+	    <parent link="front_link"/>
+	    <child link="camera_link"/>
+	  </joint>
+	  <link name="camera_link">
+	    <collision>
+	      <origin xyz="0 0 0" rpy="0 0 0"/>
+	      <geometry>
+		<box size="0.2 0.2 0.2"/>
+	      </geometry>
+	    </collision>
+	    <visual>
+	      <origin xyz="0 0 0" rpy="0 0 0"/>
+	      <geometry>
+		<box size="0.2 0.2 0.2"/>
+	      </geometry>
+	      <material name="red"/>
+	    </visual>
+	    <inertial>
+	      <mass value="1e-5" />
+	      <origin xyz="0 0 0" rpy="0 0 0"/>
+	      <inertia ixx="1e-6" ixy="0" ixz="0" iyy="1e-6" iyz="0" izz="1e-6" />
+	    </inertial>
+	  </link>
+	  <!-- GPS -->
+	  <joint name="gps_joint" type="fixed">
+	    <axis xyz="1 0 0" />
+	    <origin xyz="0.2 0.2 0.2" rpy="0 0 0"/>
+	    <parent link="front_link"/>
+	    <child link="gps_link"/>
+	  </joint>
+	  <link name="gps_link">
+	    <collision>
+	      <origin xyz="1 0 0" rpy="0 0 0"/>
+	      <geometry>
+		<box size="0.2 0.2 0.2"/>
+	      </geometry>
+	    </collision>
+	    <visual>
+	      <origin xyz="1 0 0" rpy="0 0 0"/>
+	      <geometry>
+		<box size="0.2 0.2 0.2"/>
+	      </geometry>
+	      <material name="red"/>
+	    </visual>
+	    <inertial>
+	      <mass value="1e-5" />
+	      <origin xyz="0 0 0" rpy="0 0 0"/>
+	      <inertia ixx="1e-6" ixy="0" ixz="0" iyy="1e-6" iyz="0" izz="1e-6" />
+	    </inertial>
+	  </link>
         <gazebo reference="laser_base_link">
             <material>Gazebo/Black</material>
@@ -377,9 +431,10 @@
             <material>Gazebo/Black</material>
         </gazebo>
-	<gazebo reference="gps_link">
-		<plugin name="gps" filename="libhector_gazebo_ros_gps.so">
+	<!-- GPS. It's a model type, so it needs to attach to a link, not a joint. See bodyName for where this gets attached -->
+	<gazebo>
+		<plugin name="gps_plugin" filename="libhector_gazebo_ros_gps.so">
 			<alwayson>1</alwayson>
 			<updaterate>10.0</updaterate>
-			<bodyname>basefootprint</bodyname>
+			<bodyname>gps_link</bodyname>
 			<topicname>gpsfix</topicname>
 			<velocitytopicname>gpsfixvelocity</velocitytopicname>
@@ -390,3 +445,58 @@
 		</plugin>
 	</gazebo>
+	<gazebo>
+		<plugin name="imu_plugin" filename="libhector_gazebo_ros_imu.so">
+			<alwayson>1</alwayson>
+			<updaterate>10.0</updaterate>
+			<bodyname>base_link</bodyname>
+			<topicname>imu</topicname>
+		</plugin>
+	</gazebo>
+	  <!-- camera -->
+	  <gazebo reference="camera_link">
+	    <sensor type="camera" name="camera1">
+	      <update_rate>30.0</update_rate>
+	      <camera name="head">
+		<horizontal_fov>1.3962634</horizontal_fov>
+		<image>
+		  <width>800</width>
+		  <height>800</height>
+		  <format>R8G8B8</format>
+		</image>
+		<clip>
+		  <near>0.02</near>
+		  <far>300</far>
+		</clip>
+		<noise>
+		  <type>gaussian</type>
+		  <!-- Noise is sampled independently per pixel on each frame.
+		       That pixel's noise value is added to each of its color
+		       channels, which at that point lie in the range [0,1]. -->
+		  <mean>0.0</mean>
+		  <stddev>0.007</stddev>
+		</noise>
+	      </camera>
+	      <plugin name="camera_controller" filename="libgazebo_ros_camera.so">
+		<alwaysOn>true</alwaysOn>
+		<updateRate>0.0</updateRate>
+		<cameraName>camera1</cameraName>
+		<imageTopicName>image_raw</imageTopicName>
+		<cameraInfoTopicName>camera_info</cameraInfoTopicName>
+		<frameName>camera_link_optical</frameName>
+		<!-- setting hackBaseline to anything but 0.0 will cause a misalignment
+		    between the gazebo sensor image and the frame it is supposed to
+		    be attached to -->
+		<hackBaseline>0.0</hackBaseline>
+		<distortionK1>0.0</distortionK1>
+		<distortionK2>0.0</distortionK2>
+		<distortionK3>0.0</distortionK3>
+		<distortionT1>0.0</distortionT1>
+		<distortionT2>0.0</distortionT2>
+		<CxPrime>0</CxPrime>
+		<Cx>0.0</Cx>
+		<Cy>0.0</Cy>
+		<focalLength>0.0</focalLength>
+	      </plugin>
+	    </sensor>
+	  </gazebo>
 </robot>

Commit message: Made car bigger, sensor fusion launches (but has many errors)

File: car/urdf/car.xacro (robot description, xacro)
@@ -4,9 +4,9 @@
     <xacro:property name="M_PI" value="3.1415926535897931" />
     <!-- Dimension Macros -->
-    <xacro:property name="carLength" value="0.3" />
-    <xacro:property name="carWidth" value="0.15" />
-    <xacro:property name="carHeight" value="0.1" />
-    <xacro:property name="wheelRadius" value="0.06" />
-    <xacro:property name="wheelWidth" value="0.025" />
+    <xacro:property name="carLength" value="3" />
+    <xacro:property name="carWidth" value="1.5" />
+    <xacro:property name="carHeight" value="1" />
+    <xacro:property name="wheelRadius" value="0.6" />
+    <xacro:property name="wheelWidth" value="0.05" />
     <!-- Physical Material Macros -->
     <material name="Red">
@@ -54,5 +54,5 @@
     	<parent link="base_link"/>
     	<child link="front_link"/>
-    	<origin xyz="0.16 0.0 -0.1"/>
+    	<origin xyz="1.6 0.0 -0.5"/>
     </joint>
     <link name="front_link">
@@ -64,5 +64,5 @@
         <visual>
             <geometry>
-                <box size="${carLength*0.05} ${carWidth} ${carHeight*0.05}" />
+                <box size="${carLength*0.05} ${carWidth*1.2} ${carHeight*0.05}" />
             </geometry>
             <material name="Aqua"/>
@@ -70,5 +70,5 @@
         <collision>
             <geometry>
-                <box size="${carLength*0.05} ${carWidth} ${carHeight*0.05}" />
+                <box size="${carLength*0.05} ${carWidth*1.2} ${carHeight*0.05}" />
             </geometry>
         </collision>
@@ -92,5 +92,5 @@
         </inertial>
         <visual>
-            <origin xyz="-0.02 0 0" />
+            <origin xyz="-0.2 0 0" />
             <geometry>
                 <box size="${carLength*0.1} ${carWidth*0.133} ${carHeight*0.05}" />
@@ -99,5 +99,5 @@
         </visual>
         <collision>
-            <origin xyz="0.02 0 0" />
+            <origin xyz="0.2 0 0" />
             <geometry>
                 <box size="${carLength*0.1} ${carWidth*0.133} ${carHeight*0.05}" />
@@ -114,5 +114,5 @@
         <parent link="front_link" />
         <child link="front_left_bar_link" />
-        <origin xyz="0.0 0.06 0.0" rpy="0 0 0" />
+        <origin xyz="0.0 ${carWidth*0.5} 0.0" rpy="0 0 0" />
     </joint>
     <link name="front_left_bar_link">
@@ -145,5 +145,5 @@
         <parent link="front_link" />
         <child link="front_right_bar_link" />
-        <origin xyz="0.0 -0.06 0.0" rpy="0 0 0" />
+        <origin xyz="0.0 ${carWidth*-0.5} 0.0" rpy="0 0 0" />
     </joint>
     <link name="front_right_bar_link">
@@ -237,5 +237,5 @@
         <parent link="steer_link" />
         <child link="ackermann_bar_link" />
-        <origin xyz="-0.04 0 0" rpy="0 0 0" />
+        <origin xyz="-0.4 0 0" rpy="0 0 0" />
     </joint>
     <link name="ackermann_bar_link">
@@ -268,5 +268,5 @@
         <parent link="base_link" />
         <child link="back_left_wheel_link" />
-        <origin xyz="-0.16 0.1 -0.1" rpy="0 0 0" />
+        <origin xyz="-1.6 ${carWidth*0.5} -0.5" rpy="0 0 0" />
     </joint>
     <link name="back_left_wheel_link">
@@ -298,5 +298,5 @@
         <parent link="base_link" />
         <child link="back_right_wheel_link" />
-        <origin xyz="-0.16 -0.1 -0.1" rpy="0 0 0" />
+        <origin xyz="-1.6 ${carWidth*-0.5} -0.5" rpy="0 0 0" />
     </joint>
     <link name="back_right_wheel_link">
@@ -374,6 +374,6 @@
 	  <joint name="camera_joint" type="fixed">
 	    <axis xyz="0 1 0" />
-	    <origin xyz="0.2 0.2 0.2" rpy="0 0 0"/>
-	    <parent link="front_link"/>
+	    <origin xyz="0 0 ${carHeight}" rpy="0 0 0"/>
+	    <parent link="base_link"/>
 	    <child link="camera_link"/>
 	  </joint>
@@ -401,11 +401,11 @@
 	  <joint name="gps_joint" type="fixed">
 	    <axis xyz="1 0 0" />
-	    <origin xyz="0.2 0.2 0.2" rpy="0 0 0"/>
-	    <parent link="front_link"/>
+	    <origin xyz="0 0 ${carHeight*2}" rpy="0 0 0"/>
+	    <parent link="base_link"/>
 	    <child link="gps_link"/>
 	  </joint>
 	  <link name="gps_link">
 	    <collision>
-	      <origin xyz="1 0 0" rpy="0 0 0"/>
+	      <origin xyz="0 0 0" rpy="0 0 0"/>
 	      <geometry>
 		<box size="0.2 0.2 0.2"/>
@@ -434,21 +434,21 @@
 	<gazebo>
 		<plugin name="gps_plugin" filename="libhector_gazebo_ros_gps.so">
-			<alwayson>1</alwayson>
-			<updaterate>10.0</updaterate>
-			<bodyname>gps_link</bodyname>
-			<topicname>gpsfix</topicname>
-			<velocitytopicname>gpsfixvelocity</velocitytopicname>
+			<alwaysOn>1</alwaysOn>
+			<updateRate>10.0</updateRate>
+			<bodyName>gps_link</bodyName>
+			<topicName>gps/fix</topicName>
+			<velocityTopicName>gps/fix/velocity</velocityTopicName>
 			<drift>5.0 5.0 5.0</drift>
-			<gaussiannoise>0.1 0.1 0.1</gaussiannoise>
-			<velocitydrift>0 0 0</velocitydrift>
-			<velocitygaussiannoise>0.1 0.1 0.1</velocitygaussiannoise>
+			<gaussianNoise>0.1 0.1 0.1</gaussianNoise>
+			<velocityDrift>0 0 0</velocityDrift>
+			<velocityGaussianNoise>0.1 0.1 0.1</velocityGaussianNoise>
 		</plugin>
 	</gazebo>
 	<gazebo>
 		<plugin name="imu_plugin" filename="libhector_gazebo_ros_imu.so">
-			<alwayson>1</alwayson>
-			<updaterate>10.0</updaterate>
-			<bodyname>base_link</bodyname>
-			<topicname>imu</topicname>
+			<alwaysOn>1</alwaysOn>
+			<updateRate>10.0</updateRate>
+			<bodyName>base_link</bodyName>
+			<topicName>imu/data</topicName>
 		</plugin>
 	</gazebo>

Commit message: Made car look better, working on sensor fusion

File: car/urdf/car.xacro (robot description, xacro)
@@ -324,5 +324,5 @@
     </gazebo>
         <joint name="laser_base_mount_joint" type="fixed">
-            <origin xyz="0 0 0.05" rpy="0 0 0" />
+            <origin xyz="0 0 ${carHeight}" rpy="0 0 0" />
             <parent link="base_link"/>
             <child link="laser_base_link"/>
@@ -331,5 +331,5 @@
             <inertial>
                 <mass value="0.1"/>
-                <origin xyz="0 0 0.0"/>
+                <origin xyz="0 0 ${carHeight}"/>
                 <inertia ixx="0.1" ixy="0" ixz="0" iyy="0.1" iyz="0" izz="0.1"/>
             </inertial>
@@ -373,6 +373,6 @@
 	  <!-- Camera -->
 	  <joint name="camera_joint" type="fixed">
-	    <axis xyz="0 1 0" />
-	    <origin xyz="0 0 ${carHeight}" rpy="0 0 0"/>
+	    <axis xyz="0 0 0" />
+	    <origin xyz="1.1 0 ${carHeight*0.8}" rpy="0 0 0"/>
 	    <parent link="base_link"/>
 	    <child link="camera_link"/>
@@ -382,5 +382,5 @@
 	      <origin xyz="0 0 0" rpy="0 0 0"/>
 	      <geometry>
-		<box size="0.2 0.2 0.2"/>
+		<box size="0.05 0.05 0.05"/>
 	      </geometry>
 	    </collision>
@@ -388,5 +388,5 @@
 	      <origin xyz="0 0 0" rpy="0 0 0"/>
 	      <geometry>
-		<box size="0.2 0.2 0.2"/>
+		<box size="0.05 0.05 0.05"/>
 	      </geometry>
 	      <material name="red"/>
@@ -400,6 +400,6 @@
 	  <!-- GPS -->
 	  <joint name="gps_joint" type="fixed">
-	    <axis xyz="1 0 0" />
-	    <origin xyz="0 0 ${carHeight*2}" rpy="0 0 0"/>
+	    <axis xyz="0 0 0" />
+	    <origin xyz="0 0 ${carHeight*0.65}" rpy="0 0 0"/>
 	    <parent link="base_link"/>
 	    <child link="gps_link"/>
@@ -409,13 +409,13 @@
 	      <origin xyz="0 0 0" rpy="0 0 0"/>
 	      <geometry>
-		<box size="0.2 0.2 0.2"/>
+		<box size="0.05 0.05 0.05"/>
 	      </geometry>
 	    </collision>
 	    <visual>
-	      <origin xyz="1 0 0" rpy="0 0 0"/>
+	      <origin xyz="0 0 0" rpy="0 0 0"/>
 	      <geometry>
-		<box size="0.2 0.2 0.2"/>
+		<box size="0.05 0.05 0.05"/>
 	      </geometry>
-	      <material name="red"/>
+	      <material name="green"/>
 	    </visual>
 	    <inertial>
@@ -443,4 +443,5 @@
 			<velocityDrift>0 0 0</velocityDrift>
 			<velocityGaussianNoise>0.1 0.1 0.1</velocityGaussianNoise>
+			<frameId></frameId>
 		</plugin>
 	</gazebo>

Commit message: Car model

File: car/urdf/car.xacro (robot description, xacro)
@@ -4,8 +4,8 @@
     <xacro:property name="M_PI" value="3.1415926535897931" />
     <!-- Dimension Macros -->
-    <xacro:property name="carLength" value="3" />
+    <xacro:property name="carLength" value="2" />
     <xacro:property name="carWidth" value="1.5" />
-    <xacro:property name="carHeight" value="1" />
-    <xacro:property name="wheelRadius" value="0.6" />
+    <xacro:property name="carHeight" value="0.2" />
+    <xacro:property name="wheelRadius" value="0.27" />
     <xacro:property name="wheelWidth" value="0.05" />
     <!-- Physical Material Macros -->
@@ -29,24 +29,20 @@
         <inertial>
             <mass value="0.2" />
-            <origin xyz="0 0 0" />
+            <origin xyz="0 0 0" rpy="0 0 0" />
             <inertia  ixx="0.2" ixy="0.0"  ixz="0.0"  iyy="0.2"  iyz="0.0"  izz="0.2" />
         </inertial>
         <visual>
+          <origin xyz="0 0 0" rpy="0 0 ${M_PI/2}"/>
+          <geometry>
+             <mesh filename="package://car/meshes/hybrid_body.obj" scale="0.01 0.01 0.01"/>
+          </geometry>
+        </visual>
+        <collision>
             <origin xyz="0 0 0" rpy="0 0 0" />
             <geometry>
                 <box size="${carLength} ${carWidth} ${carHeight}" />
             </geometry>
-            <material name="Red"/>
-        </visual>
-        <collision>
-            <origin xyz="0 0 0" rpy="0 0 0" />
-            <geometry>
-                <box size="${carLength} ${carWidth} ${carHeight}" />
-            </geometry>
-        </collision>
-    </link>
-    <gazebo reference="base_link">
-        <material>Gazebo/Red</material>
-    </gazebo>
+        </collision>
+    </link>
     <!-- Front link of Ackermann -->
     <!-- Joins to the Car body -->
@@ -54,5 +50,5 @@
     	<parent link="base_link"/>
     	<child link="front_link"/>
-    	<origin xyz="1.6 0.0 -0.5"/>
+    	<origin xyz="${carLength*0.7} 0 0.25" rpy="0 0 0"/>
     </joint>
     <link name="front_link">
@@ -184,20 +180,16 @@
         </inertial>
         <visual>
+            <origin xyz="0 0 0" rpy="0 0 ${M_PI/2}" />
+            <geometry>
+		     <mesh filename="package://car/meshes/wheel.obj" scale="0.01 0.01 0.01"/>
+            </geometry>
+        </visual>
+        <collision>
             <origin xyz="0 0 0" rpy="${M_PI/2} 0 0" />
             <geometry>
                 <cylinder radius="${wheelRadius}" length="${wheelWidth}" />
             </geometry>
-            <material name="Green"/>
-        </visual>
-        <collision>
-            <origin xyz="0 0 0" rpy="${M_PI/2} 0 0" />
-            <geometry>
-                <cylinder radius="${wheelRadius}" length="${wheelWidth}" />
-            </geometry>
-        </collision>
-    </link>
-    <gazebo reference="front_left_wheel_link">
-        <material>Gazebo/Green</material>
-    </gazebo>
+        </collision>
+    </link>
 	<!-- the front right wheel -->
     <joint name="front_right_wheel_joint" type="continuous" >
@@ -214,19 +206,18 @@
         </inertial>
         <visual>
+            <origin xyz="0 0 0" rpy="0 0 ${M_PI/2}" />
+	    <geometry>
+		     <mesh filename="package://car/meshes/wheel.obj" scale="0.01 0.01 0.01"/>
+	    </geometry>
+            <material name="Green"/>
+        </visual>
+        <collision>
             <origin xyz="0 0 0" rpy="${M_PI/2} 0 0" />
             <geometry>
                 <cylinder radius="${wheelRadius}" length="${wheelWidth}" />
             </geometry>
-            <material name="Green"/>
-        </visual>
-        <collision>
-            <origin xyz="0 0 0" rpy="${M_PI/2} 0 0" />
-            <geometry>
-                <cylinder radius="${wheelRadius}" length="${wheelWidth}" />
-            </geometry>
         </collision>
     </link>
     <gazebo reference="front_right_wheel_link">
-        <material>Gazebo/Green</material>
         <turnGravityOff>false</turnGravityOff>
     </gazebo>
@@ -268,5 +259,5 @@
         <parent link="base_link" />
         <child link="back_left_wheel_link" />
-        <origin xyz="-1.6 ${carWidth*0.5} -0.5" rpy="0 0 0" />
+        <origin xyz="-1.4 ${carWidth*0.5} 0.25" rpy="0 0 0" />
     </joint>
     <link name="back_left_wheel_link">
@@ -277,20 +268,16 @@
         </inertial>
         <visual>
+            <origin xyz="0 0 0" rpy="0 0 ${M_PI/2}" />
+            <geometry>
+		     <mesh filename="package://car/meshes/wheel.obj" scale="0.01 0.01 0.01"/>
+            </geometry>
+        </visual>
+        <collision>
             <origin xyz="0 0 0" rpy="${M_PI/2} 0 0" />
             <geometry>
                 <cylinder radius="${wheelRadius}" length="${wheelWidth}" />
             </geometry>
-            <material name="Black"/>
-        </visual>
-        <collision>
-            <origin xyz="0 0 0" rpy="${M_PI/2} 0 0" />
-            <geometry>
-                <cylinder radius="${wheelRadius}" length="${wheelWidth}" />
-            </geometry>
-        </collision>
-    </link>
-    <gazebo reference="back_left_wheel_link">
-        <material>Gazebo/Black</material>
-    </gazebo>
+        </collision>
+    </link>
 	<!-- the back right wheel -->
     <joint name="back_right_wheel_joint" type="continuous" >
@@ -298,5 +285,5 @@
         <parent link="base_link" />
         <child link="back_right_wheel_link" />
-        <origin xyz="-1.6 ${carWidth*-0.5} -0.5" rpy="0 0 0" />
+        <origin xyz="-1.4 ${carWidth*-0.5} 0.25" rpy="0 0 0" />
     </joint>
     <link name="back_right_wheel_link">
@@ -307,20 +294,16 @@
         </inertial>
         <visual>
+            <origin xyz="0 0 0" rpy="0 0 ${M_PI/2}" />
+            <geometry>
+		     <mesh filename="package://car/meshes/wheel.obj" scale="0.01 0.01 0.01"/>
+            </geometry>
+        </visual>
+        <collision>
             <origin xyz="0 0 0" rpy="${M_PI/2} 0 0" />
             <geometry>
                 <cylinder radius="${wheelRadius}" length="${wheelWidth}" />
             </geometry>
-            <material name="Black"/>
-        </visual>
-        <collision>
-            <origin xyz="0 0 0" rpy="${M_PI/2} 0 0" />
-            <geometry>
-                <cylinder radius="${wheelRadius}" length="${wheelWidth}" />
-            </geometry>
-        </collision>
-    </link>
-    <gazebo reference="back_right_wheel_link">
-        <material>Gazebo/Black</material>
-    </gazebo>
+        </collision>
+    </link>
         <joint name="laser_base_mount_joint" type="fixed">
             <origin xyz="0 0 ${carHeight}" rpy="0 0 0" />
@@ -510,3 +493,8 @@
     </sensor>
   </gazebo>
+<gazebo>
+  <plugin name="gazebo_ros_control" filename="libgazebo_ros_control.so">
+    <robotNamespace>/carcontrol</robotNamespace>
+  </plugin>
+</gazebo>
 </robot>

Commit message: Joint control but the car flies around

File: car/urdf/car.xacro (robot description, xacro)
@@ -27,9 +27,4 @@
     <!-- Main body -->
     <link name="base_link">
-        <inertial>
-            <mass value="0.2" />
-            <origin xyz="0 0 0" rpy="0 0 0" />
-            <inertia  ixx="0.2" ixy="0.0"  ixz="0.0"  iyy="0.2"  iyz="0.0"  izz="0.2" />
-        </inertial>
         <visual>
           <origin xyz="0 0 0" rpy="0 0 ${M_PI/2}"/>
@@ -493,8 +488,29 @@
     </sensor>
   </gazebo>
+<!--Must be in same namespace as the spawner in car_control.launch-->
 <gazebo>
   <plugin name="gazebo_ros_control" filename="libgazebo_ros_control.so">
-    <robotNamespace>/carcontrol</robotNamespace>
+    <robotNamespace>/car</robotNamespace>
   </plugin>
 </gazebo>
+<transmission name="LeftTransmission" type="SimpleTransmission">
+	<type>transmission_interface/SimpleTransmission</type>
+	<joint name="front_left_wheel_joint">
+		<hardwareInterface>hardware_interface/EffortJointInterface</hardwareInterface>
+	</joint>
+	<actuator name="LeftMotor">
+		<hardwareInterface>hardware_interface/EffortJointInterface</hardwareInterface>
+		<mechanicalReduction>1</mechanicalReduction>
+	</actuator>
+</transmission>
+<transmission name="RightTransmission" type="SimpleTransmission">
+	<type>transmission_interface/SimpleTransmission</type>
+	<joint name="front_right_wheel_joint">
+		<hardwareInterface>hardware_interface/EffortJointInterface</hardwareInterface>
+	</joint>
+	<actuator name="RightMotor">
+		<hardwareInterface>hardware_interface/EffortJointInterface</hardwareInterface>
+		<mechanicalReduction>1</mechanicalReduction>
+	</actuator>
+</transmission>
 </robot>
